Commit message: feat:加入rogmap mpc minco

File: mas2027_robot_description/urdf/mas2027_sentry.urdf (robot description, URDF)
Before this commit: robot mas2027_sentry, 5 links, 4 joints
Joints:
- removed joint base_footprint_to_base_link
- added joint base_link_to_base_footprint: type fixed, parent base_link, child base_footprint, origin xyz=0 0 -0.1 rpy=0 0 0
